Commit message: Testing

File: src/ros_kortex/kortex_move_it_config/gen3_move_it_config/config/7dof/gen3.srdf.xacro (robot description, xacro)
@@ -12,4 +12,5 @@
     <!--SUBGROUPS: Groups can also be formed by referencing to already defined group names-->
     <group name="arm">
+        <!-- <joint name="$(arg prefix)mounting_plate_joint" /> -->
         <joint name="$(arg prefix)joint_1" />
         <joint name="$(arg prefix)joint_2" />
@@ -21,5 +22,5 @@
         <joint name="$(arg prefix)end_effector" />
         <joint name="$(arg prefix)tool_frame_joint" />
-        <joint name="$(arg prefix)camera_joint" />
+        <!-- <joint name="$(arg prefix)camera_joint" /> -->
         <!-- Adapter joint -->
         <joint name="$(arg prefix)adapter_joint" />
@@ -86,6 +87,7 @@
     <disable_collisions link1="$(arg prefix)shoulder_link" link2="$(arg prefix)base_link" reason="Adjacent" />
     <!-- Mounting plate collision disable -->
-    <disable_collisions link1="$(arg prefix)mounting_plate_link" link2="$(arg prefix)adapter_link" reason="Adjacent" />
+    <disable_collisions link1="$(arg prefix)mounting_plate_link" link2="$(arg prefix)adapter_link" reason="Never" />
     <disable_collisions link1="$(arg prefix)mounting_plate_link" link2="$(arg prefix)bracelet_link" reason="Never" />
+    <disable_collisions link1="$(arg prefix)mounting_plate_link" link2="$(arg prefix)base_link" reason="Adjacent" />
     <disable_collisions link1="$(arg prefix)spherical_wrist_2_link" link2="$(arg prefix)mounting_plate_link" reason="Never" />
     <disable_collisions link1="$(arg prefix)spherical_wrist_1_link" link2="$(arg prefix)mounting_plate_link" reason="Never" />
