Commit message: URDF changes to include top plate and adapter

File: src/ros_kortex/kortex_description/robots/kortex_robot.xacro (robot description, xacro)
@@ -43,4 +43,52 @@
                 <axis xyz="0 0 0" />
             </joint>
+            <!-- Add adapter link and joint -->
+            <link name="${prefix}adapter_link">
+                <visual>
+                    <origin xyz="0 0 0" rpy="0 0 0" />
+                    <geometry>
+                    <mesh filename="package://kortex_description/arms/gen3/${dof}dof/meshes/adapter_link.stl" />
+                    </geometry>
+                    <material name="">
+                    <color rgba="0.0 0.3 0.3 1" />
+                    </material>
+                </visual>
+                <collision>
+                    <origin xyz="0 0 0" rpy="0 0 0" />
+                    <geometry>
+                    <mesh filename="package://kortex_description/arms/gen3/${dof}dof/meshes/adapter_link.stl" />
+                    </geometry>
+                </collision>
+            </link>
+            <joint name="${prefix}adapter_joint" type="fixed">
+                <origin xyz="0 0 0.003" rpy="0 0 0" />
+                <child link="${prefix}adapter_link" />
+                <parent link="${prefix}tool_frame" />
+                <axis xyz="0 0 0" />
+            </joint>
+            <!-- Add top plate link and joint -->
+            <link name="${prefix}top_plate_link">
+                <visual>
+                    <origin xyz="0 0 0" rpy="0 0 0" />
+                    <geometry>
+                    <mesh filename="package://kortex_description/arms/gen3/${dof}dof/meshes/top_plate_link.stl" />
+                    </geometry>
+                    <material name="">
+                    <color rgba="0.0 0.3 0.3 1" />
+                    </material>
+                </visual>
+                <collision>
+                    <origin xyz="0 0 0" rpy="0 0 0" />
+                    <geometry>
+                    <mesh filename="package://kortex_description/arms/gen3/${dof}dof/meshes/top_plate_link.stl" />
+                    </geometry>
+                </collision>
+            </link>
+            <joint name="${prefix}top_plate_joint" type="fixed">
+                <origin xyz="0 0 0.0165" rpy="0 0 0" />
+                <parent link="${prefix}adapter_link" />
+                <child link="${prefix}top_plate_link" />
+                <axis xyz="0 0 0" />
+            </joint>
         </xacro:if>
         <!-- Load the Gazebo transmissions and gazebo_ros_control plugin -->

File: src/ros_kortex/kortex_move_it_config/gen3_move_it_config/config/7dof/gen3.srdf.xacro (robot description, xacro)
@@ -21,4 +21,7 @@
         <joint name="$(arg prefix)end_effector" />
         <joint name="$(arg prefix)tool_frame_joint" />
+        <!-- Adapter joint -->
+        <joint name="$(arg prefix)adapter_joint" />
+        <joint name="$(arg prefix)top_plate_joint" />
     </group>
     <!--GROUP STATES: Purpose: Define a named state for a particular group, in terms of joint values. This is useful to define states like 'folded arms'-->
@@ -54,4 +57,6 @@
     <disable_collisions link1="$(arg prefix)bracelet_link" link2="$(arg prefix)spherical_wrist_1_link" reason="Never" />
     <disable_collisions link1="$(arg prefix)bracelet_link" link2="$(arg prefix)spherical_wrist_2_link" reason="Adjacent" />
+    <!-- Adapter collision disable -->
+    <disable_collisions link1="$(arg prefix)bracelet_link" link2="$(arg prefix)adapter_link" reason="Adjacent" />
     <disable_collisions link1="$(arg prefix)forearm_link" link2="$(arg prefix)half_arm_1_link" reason="Never" />
     <disable_collisions link1="$(arg prefix)forearm_link" link2="$(arg prefix)half_arm_2_link" reason="Adjacent" />

Commit message: Config changes for URDF

File: src/ros_kortex/kortex_description/robots/kortex_robot.xacro (robot description, xacro)
@@ -43,52 +43,87 @@
                 <axis xyz="0 0 0" />
             </joint>
-            <!-- Add adapter link and joint -->
-            <link name="${prefix}adapter_link">
-                <visual>
-                    <origin xyz="0 0 0" rpy="0 0 0" />
+            <xacro:if value="${not sim}">
+                <!-- Add adapter link and joint -->
+                <link name="${prefix}adapter_link">
+                    <visual>
+                        <origin xyz="0 0 0" rpy="0 0 0" />
+                        <geometry>
+                        <mesh filename="package://kortex_description/arms/gen3/${dof}dof/meshes/adapter_link.stl" />
+                        </geometry>
+                        <material name="teal">
+                        <color rgba="0.0 0.3 0.3 1" />
+                        </material>
+                    </visual>
+                    <collision>
+                        <origin xyz="0 0 0" rpy="0 0 0" />
+                        <geometry>
+                        <mesh filename="package://kortex_description/arms/gen3/${dof}dof/meshes/adapter_link.stl" />
+                        </geometry>
+                    </collision>
+                    <inertial>
+                        <mass value="0.040"/>
+                        <origin rpy="0 0 0" xyz="-0.000281 0.0 0.005605"/>
+                        <inertia
+                        ixx="200.386093e-05"
+                        ixy="0.001830e-05"
+                        ixz="-0.265552e-05"
+                        iyy="187.832535e-05"
+                        iyz="0.000163e-05"
+                        izz="355.281738e-05"/>
+                    </inertial>
+                </link>
+                <joint name="${prefix}adapter_joint" type="fixed">
+                    <origin xyz="0 0 0.003" rpy="0 0 0" />
+                    <child link="${prefix}adapter_link" />
+                    <parent link="${prefix}tool_frame" />
+                    <axis xyz="0 0 0" />
+                </joint>
+                <!-- Add top plate link and joint -->
+                <link name="${prefix}top_plate_link">
+                    <visual>
+                        <origin xyz="0 0 0" rpy="0 0 0" />
+                        <geometry>
+                        <mesh filename="package://kortex_description/arms/gen3/${dof}dof/meshes/top_plate_link.stl" />
+                        </geometry>
+                        <material name="">
+                        <color rgba="0.0 0.3 0.3 1" />
+                        </material>
+                    </visual>
+                    <collision>
+                        <origin xyz="0 0 0" rpy="0 0 0" />
+                        <geometry>
+                        <mesh filename="package://kortex_description/arms/gen3/${dof}dof/meshes/top_plate_link.stl" />
+                        </geometry>
+                    </collision>
+                </link>
+                <joint name="${prefix}top_plate_joint" type="fixed">
+                    <origin xyz="0 0 0.0165" rpy="0 0 3.14159265" />
+                    <parent link="${prefix}adapter_link" />
+                    <child link="${prefix}top_plate_link" />
+                    <axis xyz="0 0 0" />
+                </joint>
+                <!-- Add mounting plate -->
+                <link name="mounting_plate_link">
+                    <visual>
+                        <geometry>
+                            <cylinder length="0.02" radius="0.080"/>
+                        </geometry>
+                        <material name="blue">
+                            <color rgba="0 0 .8 1"/>
+                        </material>
+                    </visual>
+                <collision>
                     <geometry>
-                    <mesh filename="package://kortex_description/arms/gen3/${dof}dof/meshes/adapter_link.stl" />
-                    </geometry>
-                    <material name="">
-                    <color rgba="0.0 0.3 0.3 1" />
-                    </material>
-                </visual>
-                <collision>
-                    <origin xyz="0 0 0" rpy="0 0 0" />
-                    <geometry>
-                    <mesh filename="package://kortex_description/arms/gen3/${dof}dof/meshes/adapter_link.stl" />
+                    <cylinder length="0.02" radius="0.080"/>
                     </geometry>
                 </collision>
-            </link>
-            <joint name="${prefix}adapter_joint" type="fixed">
-                <origin xyz="0 0 0.003" rpy="0 0 0" />
-                <child link="${prefix}adapter_link" />
-                <parent link="${prefix}tool_frame" />
-                <axis xyz="0 0 0" />
-            </joint>
-            <!-- Add top plate link and joint -->
-            <link name="${prefix}top_plate_link">
-                <visual>
+                </link>
+                <joint name="${prefix}mounting_plate_joint" type="fixed">
                     <origin xyz="0 0 0" rpy="0 0 0" />
-                    <geometry>
-                    <mesh filename="package://kortex_description/arms/gen3/${dof}dof/meshes/top_plate_link.stl" />
-                    </geometry>
-                    <material name="">
-                    <color rgba="0.0 0.3 0.3 1" />
-                    </material>
-                </visual>
-                <collision>
-                    <origin xyz="0 0 0" rpy="0 0 0" />
-                    <geometry>
-                    <mesh filename="package://kortex_description/arms/gen3/${dof}dof/meshes/top_plate_link.stl" />
-                    </geometry>
-                </collision>
-            </link>
-            <joint name="${prefix}top_plate_joint" type="fixed">
-                <origin xyz="0 0 0.0165" rpy="0 0 0" />
-                <parent link="${prefix}adapter_link" />
-                <child link="${prefix}top_plate_link" />
-                <axis xyz="0 0 0" />
-            </joint>
+                    <parent link="${prefix}base_link" />
+                    <child link="${prefix}mounting_plate_link" />
+                    <axis xyz="0 0 0" />
+                </joint>
+            </xacro:if>
         </xacro:if>
         <!-- Load the Gazebo transmissions and gazebo_ros_control plugin -->

File: src/ros_kortex/kortex_move_it_config/gen3_move_it_config/config/7dof/gen3.srdf.xacro (robot description, xacro)
@@ -59,4 +59,11 @@
     <!-- Adapter collision disable -->
     <disable_collisions link1="$(arg prefix)bracelet_link" link2="$(arg prefix)adapter_link" reason="Adjacent" />
+    <disable_collisions link1="$(arg prefix)spherical_wrist_2_link" link2="$(arg prefix)adapter_link" reason="Never" />
+    <disable_collisions link1="$(arg prefix)spherical_wrist_1_link" link2="$(arg prefix)adapter_link" reason="Never" />
+    <disable_collisions link1="$(arg prefix)forearm_link" link2="$(arg prefix)adapter_link" reason="Never" />
+    <disable_collisions link1="$(arg prefix)half_arm_2_link" link2="$(arg prefix)adapter_link" reason="Never" />
+    <disable_collisions link1="$(arg prefix)half_arm_1_link" link2="$(arg prefix)adapter_link" reason="Never" />
+    <disable_collisions link1="$(arg prefix)shoulder_link" link2="$(arg prefix)adapter_link" reason="Never" />
+    <disable_collisions link1="$(arg prefix)base_link" link2="$(arg prefix)adapter_link" reason="Never" />
     <disable_collisions link1="$(arg prefix)forearm_link" link2="$(arg prefix)half_arm_1_link" reason="Never" />
     <disable_collisions link1="$(arg prefix)forearm_link" link2="$(arg prefix)half_arm_2_link" reason="Adjacent" />
@@ -77,4 +84,11 @@
     <disable_collisions link1="$(arg prefix)shoulder_link" link2="$(arg prefix)spherical_wrist_2_link" reason="Never" />
     <disable_collisions link1="$(arg prefix)shoulder_link" link2="$(arg prefix)base_link" reason="Adjacent" />
+    <!-- Mounting plate collision disable -->
+    <disable_collisions link1="$(arg prefix)mounting_plate_link" link2="$(arg prefix)adapter_link" reason="Adjacent" />
+    <disable_collisions link1="$(arg prefix)mounting_plate_link" link2="$(arg prefix)bracelet_link" reason="Never" />
+    <disable_collisions link1="$(arg prefix)spherical_wrist_2_link" link2="$(arg prefix)mounting_plate_link" reason="Never" />
+    <disable_collisions link1="$(arg prefix)spherical_wrist_1_link" link2="$(arg prefix)mounting_plate_link" reason="Never" />
+    <disable_collisions link1="$(arg prefix)forearm_link" link2="$(arg prefix)mounting_plate_link" reason="Never" />
+    <disable_collisions link1="$(arg prefix)shoulder_link" link2="$(arg prefix)base_link" reason="Adjacent" />
     <disable_collisions link1="$(arg prefix)spherical_wrist_1_link" link2="$(arg prefix)spherical_wrist_2_link" reason="Adjacent" />
 </robot>

Commit message: acquire data sphere working with camera link frame

File: src/ros_kortex/kortex_description/robots/kortex_robot.xacro (robot description, xacro)
@@ -43,4 +43,13 @@
                 <axis xyz="0 0 0" />
             </joint>
+            <!-- Define a joint with the tool frame as a parent called camera_joint -->
+            <joint name="${prefix}camera_joint" type="fixed">
+                <origin xyz="0.0 0.1 0.04" rpy="${-pi/2} 0 0" />
+                <parent link="${prefix}tool_frame" />
+                <child link="${prefix}camera_link" />
+                <axis xyz="0 0 0" />
+            </joint>
+            <!-- Define camera_link -->
+            <link name="${prefix}camera_link"/>
             <xacro:if value="${not sim}">
                 <!-- Add adapter link and joint -->

File: src/ros_kortex/kortex_move_it_config/gen3_move_it_config/config/7dof/gen3.srdf.xacro (robot description, xacro)
@@ -21,4 +21,5 @@
         <joint name="$(arg prefix)end_effector" />
         <joint name="$(arg prefix)tool_frame_joint" />
+        <joint name="$(arg prefix)camera_joint" />
         <!-- Adapter joint -->
         <joint name="$(arg prefix)adapter_joint" />

Commit message: Latest changes

File: src/ros_kortex/kortex_description/robots/kortex_robot.xacro (robot description, xacro)
@@ -91,7 +91,7 @@
                 <link name="${prefix}top_plate_link">
                     <visual>
-                        <origin xyz="0 0 0" rpy="0 0 0" />
+                        <origin xyz="0 0 0" rpy="0 0 0.003" />
                         <geometry>
-                        <mesh filename="package://kortex_description/arms/gen3/${dof}dof/meshes/top_plate_link.stl" />
+                        <box size="0.2 0.2 0.003"/>
                         </geometry>
                         <material name="">

File: src/ros_kortex/kortex_move_it_config/gen3_move_it_config/config/7dof/gen3.srdf.xacro (robot description, xacro)
@@ -55,4 +55,13 @@
         <joint name="$(arg prefix)joint_7" value="0" />
     </group_state>
+    <group_state name="compatible_vertical" group="arm">
+        <joint name="$(arg prefix)joint_1" value="0" />
+        <joint name="$(arg prefix)joint_2" value="0" />
+        <joint name="$(arg prefix)joint_3" value="3.14" />
+        <joint name="$(arg prefix)joint_4" value="0" />
+        <joint name="$(arg prefix)joint_5" value="0" />
+        <joint name="$(arg prefix)joint_6" value="0" />
+        <joint name="$(arg prefix)joint_7" value="1.57" />
+    </group_state>
     <!--DISABLE COLLISIONS: By default it is assumed that any link of the robot could potentially come into collision with any other link in the robot. This tag disables collision checking between a specified pair of links. -->
     <disable_collisions link1="$(arg prefix)bracelet_link" link2="$(arg prefix)forearm_link" reason="Never" />

Commit message: STL files added for RGB stereo plates

File: src/ros_kortex/kortex_description/robots/kortex_robot.xacro (robot description, xacro)
@@ -58,5 +58,5 @@
                         <origin xyz="0 0 0" rpy="0 0 0" />
                         <geometry>
-                        <mesh filename="package://kortex_description/arms/gen3/${dof}dof/meshes/adapter_link.stl" />
+                        <mesh filename="package://kortex_description/arms/gen3/${dof}dof/meshes/adapter_link_LR.stl" />
                         </geometry>
                         <material name="teal">
@@ -67,18 +67,7 @@
                         <origin xyz="0 0 0" rpy="0 0 0" />
                         <geometry>
-                        <mesh filename="package://kortex_description/arms/gen3/${dof}dof/meshes/adapter_link.stl" />
+                        <mesh filename="package://kortex_description/arms/gen3/${dof}dof/meshes/adapter_link_LR.stl" />
                         </geometry>
                     </collision>
-                    <inertial>
-                        <mass value="0.040"/>
-                        <origin rpy="0 0 0" xyz="-0.000281 0.0 0.005605"/>
-                        <inertia
-                        ixx="200.386093e-05"
-                        ixy="0.001830e-05"
-                        ixz="-0.265552e-05"
-                        iyy="187.832535e-05"
-                        iyz="0.000163e-05"
-                        izz="355.281738e-05"/>
-                    </inertial>
                 </link>
                 <joint name="${prefix}adapter_joint" type="fixed">
@@ -91,16 +80,16 @@
                 <link name="${prefix}top_plate_link">
                     <visual>
-                        <origin xyz="0 0 0" rpy="0 0 0.003" />
+                        <origin xyz="0 0 0" rpy="0 0 0" />
                         <geometry>
-                        <box size="0.2 0.2 0.003"/>
+                            <mesh filename="package://kortex_description/arms/gen3/${dof}dof/meshes/small_top_plate_link_LR.stl" />
                         </geometry>
                         <material name="">
-                        <color rgba="0.0 0.3 0.3 1" />
+                            <color rgba="0.0 0.3 0.3 1" />
                         </material>
                     </visual>
                     <collision>
-                        <origin xyz="0 0 0" rpy="0 0 0" />
+                        <origin xyz="0 0 0.0015" rpy="0 0 0" />
                         <geometry>
-                        <mesh filename="package://kortex_description/arms/gen3/${dof}dof/meshes/top_plate_link.stl" />
+                            <box size="0.1 0.075 0.003"/>
                         </geometry>
                     </collision>

File: src/ros_kortex/kortex_move_it_config/gen3_move_it_config/config/7dof/gen3.srdf.xacro (robot description, xacro)
@@ -22,8 +22,8 @@
         <joint name="$(arg prefix)end_effector" />
         <joint name="$(arg prefix)tool_frame_joint" />
-        <!-- <joint name="$(arg prefix)camera_joint" /> -->
         <!-- Adapter joint -->
-        <joint name="$(arg prefix)adapter_joint" />
-        <joint name="$(arg prefix)top_plate_joint" />
+        <!-- <joint name="$(arg prefix)adapter_joint" />
+        <joint name="$(arg prefix)top_plate_joint" /> -->
+        <joint name="$(arg prefix)camera_joint" />
     </group>
     <!--GROUP STATES: Purpose: Define a named state for a particular group, in terms of joint values. This is useful to define states like 'folded arms'-->
