Commit message: Add SRDF collision disable (unfinished)

File: src/ros_kortex/kortex_description/robots/kortex_robot.xacro (robot description, xacro)
@@ -97,4 +97,26 @@
                     <axis xyz="0 0 0" />
                 </joint>
+                <!-- Add extrusion parts -->
+                <link name="extrusion_link">
+                    <visual>
+                        <geometry>
+                            <box size="0.40 0.3 0.045"/>
+                        </geometry>
+                        <material name="">
+                            <color rgba="0.6 0.6 0.6 1"/>
+                        </material>
+                    </visual>
+                    <collision>
+                        <geometry>
+                            <box size="0.40 0.3 0.045"/>
+                        </geometry>
+                    </collision>
+                </link>
+                <joint name="${prefix}extrusion_joint" type="fixed">
+                    <origin xyz="0.05 0 -0.024" rpy="0 0 0" />
+                    <parent link="${prefix}kinova_plate_link" />
+                    <child link="${prefix}extrusion_link" />
+                    <axis xyz="0 0 0" />
+                </joint>
                 <!-- Add adapter link and joint -->
                 <link name="${prefix}adapter_link">
@@ -116,5 +138,5 @@
                 </link>
                 <joint name="${prefix}adapter_joint" type="fixed">
-                    <origin xyz="0 0 0.003" rpy="0 0 0" />
+                    <origin xyz="0 0 0.003" rpy="0 0 ${pi}" />
                     <child link="${prefix}adapter_link" />
                     <parent link="${prefix}tool_frame" />
@@ -218,5 +240,5 @@
                 <!-- Add cameras -->
                 <xacro:include filename="$(find flir_camera_description)/urdf/flir_blackflys.urdf.xacro" />
-                <xacro:flir_blackflys name="camLeft" frame="${prefix}left_camera_link" />
+                <xacro:flir_blackflys name="left_camera" frame="${prefix}left_camera_link" />
                 <joint name="${prefix}left_camera_joint" type="fixed">
                     <origin xyz="0.02 0.01565 0" rpy="${pi} 0 ${pi/2}" />
@@ -225,5 +247,5 @@
                     <axis xyz="0 0 0" />
                 </joint>
-                <xacro:flir_blackflys name="camRight" frame="${prefix}right_camera_link" />
+                <xacro:flir_blackflys name="right_camera" frame="${prefix}right_camera_link" />
                 <joint name="${prefix}right_camera_joint" type="fixed">
                     <origin xyz="-0.02 0.01565 0" rpy="${pi} 0 ${pi/2}" />

File: src/ros_kortex/kortex_move_it_config/gen3_move_it_config/config/7dof/gen3.srdf.xacro (robot description, xacro)
@@ -80,4 +80,26 @@
     <disable_collisions link1="$(arg prefix)shoulder_link" link2="$(arg prefix)adapter_link" reason="Never" />
     <disable_collisions link1="$(arg prefix)base_link" link2="$(arg prefix)adapter_link" reason="Never" />
+    <!-- Disable collisions for the left camera links and the lenses -->
+    <disable_collisions link1="$(arg prefix)left_camera_link" link2="$(arg prefix)left_camera_link_lens" reason="Adjacent" />
+    <disable_collisions link1="$(arg prefix)left_camera_link" link2="$(arg prefix)left_camera_link_optical" reason="Adjacent" />
+    <disable_collisions link1="$(arg prefix)left_camera_link_lens" link2="$(arg prefix)left_camera_link_optical" reason="Adjacent" />
+    <!-- Disable collisions for the right camera links and lenses -->
+    <disable_collisions link1="$(arg prefix)right_camera_link" link2="$(arg prefix)right_camera_link_lens" reason="Adjacent" />
+    <disable_collisions link1="$(arg prefix)right_camera_link" link2="$(arg prefix)right_camera_link_optical" reason="Adjacent" />
+    <disable_collisions link1="$(arg prefix)right_camera_link_lens" link2="$(arg prefix)right_camera_link_optical" reason="Adjacent" />
+    <!-- Disable collisions for the plates and cameras-->
+    <disable_collisions link1="$(arg prefix)camera_plate_link" link2="$(arg prefix)top_plate_link" reason="Never" />
+    <disable_collisions link1="$(arg prefix)camera_plate_link" link2="$(arg prefix)left_camera_link" reason="Adjacent" />
+    <disable_collisions link1="$(arg prefix)camera_plate_link" link2="$(arg prefix)right_camera_link" reason="Adjacent" />
+    <disable_collisions link1="$(arg prefix)top_plate_link" link2="$(arg prefix)left_camera_link" reason="Never" />
+    <disable_collisions link1="$(arg prefix)top_plate_link" link2="$(arg prefix)right_camera_link" reason="Never" />
+    <!-- Mounting plate collision disable -->
+    <disable_collisions link1="$(arg prefix)mounting_plate_link" link2="$(arg prefix)adapter_link" reason="Never" />
+    <disable_collisions link1="$(arg prefix)mounting_plate_link" link2="$(arg prefix)bracelet_link" reason="Never" />
+    <disable_collisions link1="$(arg prefix)mounting_plate_link" link2="$(arg prefix)base_link" reason="Adjacent" />
+    <disable_collisions link1="$(arg prefix)spherical_wrist_2_link" link2="$(arg prefix)mounting_plate_link" reason="Never" />
+    <disable_collisions link1="$(arg prefix)spherical_wrist_1_link" link2="$(arg prefix)mounting_plate_link" reason="Never" />
+    <disable_collisions link1="$(arg prefix)forearm_link" link2="$(arg prefix)mounting_plate_link" reason="Never" />
+    <disable_collisions link1="$(arg prefix)kinova_plate_link" link2="$(arg prefix)mounting_plate_link" reason="Never" />
     <disable_collisions link1="$(arg prefix)forearm_link" link2="$(arg prefix)half_arm_1_link" reason="Never" />
     <disable_collisions link1="$(arg prefix)forearm_link" link2="$(arg prefix)half_arm_2_link" reason="Adjacent" />
@@ -98,11 +120,4 @@
     <disable_collisions link1="$(arg prefix)shoulder_link" link2="$(arg prefix)spherical_wrist_2_link" reason="Never" />
     <disable_collisions link1="$(arg prefix)shoulder_link" link2="$(arg prefix)base_link" reason="Adjacent" />
-    <!-- Mounting plate collision disable -->
-    <disable_collisions link1="$(arg prefix)mounting_plate_link" link2="$(arg prefix)adapter_link" reason="Never" />
-    <disable_collisions link1="$(arg prefix)mounting_plate_link" link2="$(arg prefix)bracelet_link" reason="Never" />
-    <disable_collisions link1="$(arg prefix)mounting_plate_link" link2="$(arg prefix)base_link" reason="Adjacent" />
-    <disable_collisions link1="$(arg prefix)spherical_wrist_2_link" link2="$(arg prefix)mounting_plate_link" reason="Never" />
-    <disable_collisions link1="$(arg prefix)spherical_wrist_1_link" link2="$(arg prefix)mounting_plate_link" reason="Never" />
-    <disable_collisions link1="$(arg prefix)forearm_link" link2="$(arg prefix)mounting_plate_link" reason="Never" />
     <disable_collisions link1="$(arg prefix)shoulder_link" link2="$(arg prefix)base_link" reason="Adjacent" />
     <disable_collisions link1="$(arg prefix)spherical_wrist_1_link" link2="$(arg prefix)spherical_wrist_2_link" reason="Adjacent" />
