Commit message: Add cameras to URDF

File: src/flir_camera_driver/flir_camera_description/urdf/flir_blackflys.urdf.xacro (robot description, xacro)
@@ -20,5 +20,8 @@
                 <mesh filename="package://flir_camera_description/meshes/flir_blackflys.stl"/>
             </geometry>
-            <material name="dark_grey" />
+            <material name="">
+                <color rgba="0.1 0.1 0.1 1" />
+            </material>
+            <!-- <material name="dark_grey" /> -->
         </visual>
         <collision>
@@ -39,5 +42,8 @@
             <cylinder radius="${lens_r}" length="${lens_h}"/>
             </geometry>
-            <material name="dark_grey" />
+            <material name="">
+                <color rgba="0.2 0.2 0.2 1" />
+            </material>
+            <!-- <material name="dark_grey" /> -->
         </visual>
         <collision>

File: src/ros_kortex/kortex_description/robots/kortex_robot.xacro (robot description, xacro)
@@ -53,4 +53,48 @@
             <link name="${prefix}camera_link"/>
             <xacro:if value="${not sim}">
+                <!-- Add mounting plate -->
+                <link name="mounting_plate_link">
+                    <visual>
+                        <geometry>
+                            <cylinder length="0.02" radius="0.080"/>
+                        </geometry>
+                        <material name="">
+                            <color rgba="0.15 0.15 0.15 1"/>
+                        </material>
+                    </visual>
+                    <collision>
+                        <geometry>
+                            <cylinder length="0.02" radius="0.080"/>
+                        </geometry>
+                    </collision>
+                </link>
+                <joint name="${prefix}mounting_plate_joint" type="fixed">
+                    <origin xyz="0 0 -0.01" rpy="0 0 0" />
+                    <parent link="${prefix}base_link" />
+                    <child link="${prefix}mounting_plate_link" />
+                    <axis xyz="0 0 0" />
+                </joint>
+                <!-- Add Kinova plate -->
+                <link name="kinova_plate_link">
+                    <visual>
+                        <geometry>
+                            <box size="0.3 0.3 0.003"/>
+                        </geometry>
+                        <material name="">
+                            <color rgba="0.6 0.6 0.6 1"/>
+                        </material>
+                    </visual>
+                <collision>
+                    <geometry>
+                    <box size="0.3 0.3 0.003"/>
+                    </geometry>
+                </collision>
+                </link>
+                <joint name="${prefix}kinova_plate_joint" type="fixed">
+                    <origin xyz="0 0 -0.013" rpy="0 0 0" />
+                    <parent link="${prefix}mounting_plate_link" />
+                    <child link="${prefix}kinova_plate_link" />
+                    <axis xyz="0 0 0" />
+                </joint>
                 <!-- Add adapter link and joint -->
                 <link name="${prefix}adapter_link">
@@ -61,5 +105,5 @@
                         </geometry>
                         <material name="teal">
-                        <color rgba="0.0 0.3 0.3 1" />
+                        <color rgba="0.15 0.15 0.15 1" />
                         </material>
                     </visual>
@@ -96,29 +140,94 @@
                 </link>
                 <joint name="${prefix}top_plate_joint" type="fixed">
-                    <origin xyz="0 0 0.0165" rpy="0 0 3.14159265" />
+                    <origin xyz="0 0 0.0165" rpy="0 0 ${pi}" />
                     <parent link="${prefix}adapter_link" />
                     <child link="${prefix}top_plate_link" />
                     <axis xyz="0 0 0" />
                 </joint>
-                <!-- Add mounting plate -->
-                <link name="mounting_plate_link">
-                    <visual>
-                        <geometry>
-                            <cylinder length="0.02" radius="0.080"/>
-                        </geometry>
-                        <material name="blue">
-                            <color rgba="0 0 .8 1"/>
-                        </material>
-                    </visual>
-                <collision>
-                    <geometry>
-                    <cylinder length="0.02" radius="0.080"/>
-                    </geometry>
-                </collision>
-                </link>
-                <joint name="${prefix}mounting_plate_joint" type="fixed">
+                <!-- Add side brackets -->
+                <link name="${prefix}right_side_bracket_link">
+                    <visual>
+                        <origin xyz="-0.035 0 0.028" rpy="${-pi/2} 0 ${pi/2} " />
+                        <geometry>
+                            <mesh filename="package://kortex_description/arms/gen3/${dof}dof/meshes/side_bracket_link_LR.stl" />
+                        </geometry>
+                        <material name="">
+                            <color rgba="0.8 0.8 0.8 1"/>
+                        </material>
+                    </visual>
+                    <collision>
+                        <origin xyz="-0.0425 0 0.028" rpy="${pi/2} 0 ${-pi/2} "  />
+                        <geometry>
+                            <box size="0.075 0.05 0.015"/>
+                        </geometry>
+                    </collision>
+                </link>
+                <joint name="${prefix}right_side_bracket_joint" type="fixed">
                     <origin xyz="0 0 0" rpy="0 0 0" />
-                    <parent link="${prefix}base_link" />
-                    <child link="${prefix}mounting_plate_link" />
+                    <parent link="${prefix}top_plate_link" />
+                    <child link="${prefix}right_side_bracket_link" />
+                    <axis xyz="0 0 0" />
+                </joint>
+                <link name="${prefix}left_side_bracket_link">
+                    <visual>
+                        <origin xyz="0.035 0 0.028" rpy="${-pi/2} 0 ${-pi/2} " />
+                        <geometry>
+                            <mesh filename="package://kortex_description/arms/gen3/${dof}dof/meshes/side_bracket_link_LR.stl" />
+                        </geometry>
+                        <material name="">
+                            <color rgba="0.8 0.8 0.8 1"/>
+                        </material>
+                    </visual>
+                    <collision>
+                        <origin xyz="0.0425 0 0.028" rpy="${pi/2} 0 ${pi/2} "  />
+                        <geometry>
+                            <box size="0.075 0.05 0.015"/>
+                        </geometry>
+                    </collision>
+                </link>
+                <joint name="${prefix}left_side_bracket_joint" type="fixed">
+                    <origin xyz="0 0 0" rpy="0 0 0" />
+                    <parent link="${prefix}top_plate_link" />
+                    <child link="${prefix}left_side_bracket_link" />
+                    <axis xyz="0 0 0" />
+                </joint>
+                <!-- Add Camera plate -->
+                <link name="${prefix}camera_plate_link">
+                    <visual>
+                        <origin xyz="0 0 0" rpy="0 0 0" />
+                        <geometry>
+                            <mesh filename="package://kortex_description/arms/gen3/${dof}dof/meshes/small_camera_plate_link_LR.stl" />
+                        </geometry>
+                        <material name="">
+                            <color rgba="0.0 0.3 0.3 1" />
+                        </material>
+                    </visual>
+                    <collision>
+                        <origin xyz="0 0 0.0015" rpy="0 0 0" />
+                        <geometry>
+                            <box size="0.1 0.075 0.003"/>
+                        </geometry>
+                    </collision>
+                </link>
+                <joint name="${prefix}camera_plate_joint" type="fixed">
+                    <origin xyz="0 0 0.053" rpy="0 0 0" />
+                    <parent link="${prefix}top_plate_link" />
+                    <child link="${prefix}camera_plate_link" />
+                    <axis xyz="0 0 0" />
+                </joint>
+                <!-- Add cameras -->
+                <xacro:include filename="$(find flir_camera_description)/urdf/flir_blackflys.urdf.xacro" />
+                <xacro:flir_blackflys name="camLeft" frame="${prefix}left_camera_link" />
+                <joint name="${prefix}left_camera_joint" type="fixed">
+                    <origin xyz="0.02 0.01565 0" rpy="${pi} 0 ${pi/2}" />
+                    <parent link="${prefix}camera_plate_link" />
+                    <child link="${prefix}left_camera_link" />
+                    <axis xyz="0 0 0" />
+                </joint>
+                <xacro:flir_blackflys name="camRight" frame="${prefix}right_camera_link" />
+                <joint name="${prefix}right_camera_joint" type="fixed">
+                    <origin xyz="-0.02 0.01565 0" rpy="${pi} 0 ${pi/2}" />
+                    <parent link="${prefix}camera_plate_link" />
+                    <child link="${prefix}right_camera_link" />
                     <axis xyz="0 0 0" />
                 </joint>

File: src/ros_kortex/kortex_move_it_config/gen3_move_it_config/config/7dof/gen3.srdf.xacro (robot description, xacro)
@@ -22,8 +22,11 @@
         <joint name="$(arg prefix)end_effector" />
         <joint name="$(arg prefix)tool_frame_joint" />
-        <!-- Adapter joint -->
-        <!-- <joint name="$(arg prefix)adapter_joint" />
-        <joint name="$(arg prefix)top_plate_joint" /> -->
-        <joint name="$(arg prefix)camera_joint" />
+        <joint name="$(arg prefix)adapter_joint" />
+        <joint name="$(arg prefix)top_plate_joint" />
+        <joint name="$(arg prefix)camera_plate_joint"/>
+        <joint name="$(arg prefix)left_camera_joint"/>
+        <joint name="$(arg prefix)left_camera_link_lens_joint"/>
+        <joint name="$(arg prefix)left_camera_link_optical_joint"/>
+        <!-- <joint name="$(arg prefix)camera_joint" /> -->
     </group>
     <!--GROUP STATES: Purpose: Define a named state for a particular group, in terms of joint values. This is useful to define states like 'folded arms'-->
