Commit message: Testing

File: src/flir_camera_driver/flir_camera_description/urdf/flir_blackflys.urdf.xacro (robot description, xacro)
@@ -61,5 +61,6 @@
         </joint>
         <joint name="${frame}_optical_joint" type="fixed">
-        <origin xyz="${lens_h} 0 0" rpy="-1.570796 0 -1.570796" />
+        <!-- Change made here compared to original rpy -pi/2 0 -pi/2 -->
+        <origin xyz="${lens_h} 0 0" rpy="${pi/2} 0 ${pi/2}" />
         <parent link="${frame}_lens" />
         <child link="${frame}_optical" />

File: src/ros_kortex/kortex_description/arms/gen3/7dof/urdf/gen3_macro.xacro (robot description, xacro)
@@ -5,9 +5,10 @@
   <xacro:macro name="load_arm" params="parent:='' dof vision prefix *origin">
       <link name="${prefix}base_link">
-        <inertial>
+      <!-- Comment out inertial setting as this is the world root -->
+        <!-- <inertial>
           <origin xyz="-0.000648 -0.000166 0.084487" rpy="0 0 0" />
           <mass value="1.697" />
           <inertia ixx="0.004622" ixy="9E-06" ixz="6E-05" iyy="0.004495" iyz="9E-06" izz="0.002079" />
-        </inertial>
+        </inertial> -->
         <visual>
           <origin xyz="0 0 0" rpy="0 0 0" />
@@ -50,10 +51,84 @@
     <joint
       name="${prefix}joint_1"
+      type="revolute">
+      <origin xyz="0 0 0.15643" rpy="3.1416 2.7629E-18 -4.9305E-36" />
+      <parent
+        link="${prefix}base_link" />
+      <child
+        link="${prefix}shoulder_link" />
+      <axis
+        xyz="0 0 1" />
+      <limit
+        lower="-0.55"
+        upper="0.55"
+        effort="39"
+        velocity="1.3963" />
+      <!--  changed from continuous to revolute -->
+    </joint>
+    <link name="${prefix}half_arm_1_link">
+      <inertial>
+        <origin xyz="-4.4E-05 -0.09958 -0.013278" rpy="0 0 0" />
+        <mass value="1.1636" />
+        <inertia ixx="0.011088" ixy="5E-06" ixz="0" iyy="0.001072" iyz="-0.000691" izz="0.011255" />
+      </inertial>
+      <visual>
+        <origin xyz="0 0 0" rpy="0 0 0" />
+        <geometry>
+          <mesh filename="package://kortex_description/arms/gen3/${dof}dof/meshes/half_arm_1_link.STL" />
+        </geometry>
+        <material name="">
+          <color rgba="0.75294 0.75294 0.75294 1" />
+        </material>
+      </visual>
+      <collision>
+        <origin xyz="0 0 0" rpy="0 0 0" />
+        <geometry>
+          <mesh filename="package://kortex_description/arms/gen3/${dof}dof/meshes/half_arm_1_link.STL" />
+        </geometry>
+      </collision>
+    </link>
+    <joint
+      name="${prefix}joint_2"
+      type="revolute">
+      <origin xyz="0 0.005375 -0.12838" rpy="1.5708 2.1343E-17 -1.1102E-16" />
+      <parent
+        link="${prefix}shoulder_link" />
+      <child
+        link="${prefix}half_arm_1_link" />
+      <axis
+        xyz="0 0 1" />
+        <!-- Changed bounds to +-pi/2 from +-2.41 -->
+      <limit lower="${-pi/2}" upper="${pi/2}" effort="39" velocity="1.3963" />
+    </joint>
+    <link name="${prefix}half_arm_2_link">
+      <inertial>
+        <origin xyz="-4.4E-05 -0.006641 -0.117892" rpy="0 0 0" />
+        <mass value="1.1636" />
+        <inertia ixx="0.010932" ixy="0" ixz="-7E-06" iyy="0.011127" iyz="0.000606" izz="0.001043" />
+      </inertial>
+      <visual>
+        <origin xyz="0 0 0" rpy="0 0 0" />
+        <geometry>
+          <mesh filename="package://kortex_description/arms/gen3/${dof}dof/meshes/half_arm_2_link.STL" />
+        </geometry>
+        <material name="">
+          <color rgba="0.75294 0.75294 0.75294 1" />
+        </material>
+      </visual>
+      <collision>
+        <origin xyz="0 0 0" rpy="0 0 0" />
+        <geometry>
+          <mesh filename="package://kortex_description/arms/gen3/${dof}dof/meshes/half_arm_2_link.STL" />
+        </geometry>
+      </collision>
+    </link>
+    <joint
+      name="${prefix}joint_3"
       type="continuous">
-      <origin xyz="0 0 0.15643" rpy="3.1416 2.7629E-18 -4.9305E-36" />
-      <parent
-        link="${prefix}base_link" />
-      <child
-        link="${prefix}shoulder_link" />
+      <origin xyz="0 -0.21038 -0.006375" rpy="-1.5708 1.2326E-32 -2.9122E-16" />
+      <parent
+        link="${prefix}half_arm_1_link" />
+      <child
+        link="${prefix}half_arm_2_link" />
       <axis
         xyz="0 0 1" />
@@ -62,74 +137,4 @@
         velocity="1.3963" />
     </joint>
-    <link name="${prefix}half_arm_1_link">
-      <inertial>
-        <origin xyz="-4.4E-05 -0.09958 -0.013278" rpy="0 0 0" />
-        <mass value="1.1636" />
-        <inertia ixx="0.011088" ixy="5E-06" ixz="0" iyy="0.001072" iyz="-0.000691" izz="0.011255" />
-      </inertial>
-      <visual>
-        <origin xyz="0 0 0" rpy="0 0 0" />
-        <geometry>
-          <mesh filename="package://kortex_description/arms/gen3/${dof}dof/meshes/half_arm_1_link.STL" />
-        </geometry>
-        <material name="">
-          <color rgba="0.75294 0.75294 0.75294 1" />
-        </material>
-      </visual>
-      <collision>
-        <origin xyz="0 0 0" rpy="0 0 0" />
-        <geometry>
-          <mesh filename="package://kortex_description/arms/gen3/${dof}dof/meshes/half_arm_1_link.STL" />
-        </geometry>
-      </collision>
-    </link>
-    <joint
-      name="${prefix}joint_2"
-      type="revolute">
-      <origin xyz="0 0.005375 -0.12838" rpy="1.5708 2.1343E-17 -1.1102E-16" />
-      <parent
-        link="${prefix}shoulder_link" />
-      <child
-        link="${prefix}half_arm_1_link" />
-      <axis
-        xyz="0 0 1" />
-      <limit lower="-2.41" upper="2.41" effort="39" velocity="1.3963" />
-    </joint>
-    <link name="${prefix}half_arm_2_link">
-      <inertial>
-        <origin xyz="-4.4E-05 -0.006641 -0.117892" rpy="0 0 0" />
-        <mass value="1.1636" />
-        <inertia ixx="0.010932" ixy="0" ixz="-7E-06" iyy="0.011127" iyz="0.000606" izz="0.001043" />
-      </inertial>
-      <visual>
-        <origin xyz="0 0 0" rpy="0 0 0" />
-        <geometry>
-          <mesh filename="package://kortex_description/arms/gen3/${dof}dof/meshes/half_arm_2_link.STL" />
-        </geometry>
-        <material name="">
-          <color rgba="0.75294 0.75294 0.75294 1" />
-        </material>
-      </visual>
-      <collision>
-        <origin xyz="0 0 0" rpy="0 0 0" />
-        <geometry>
-          <mesh filename="package://kortex_description/arms/gen3/${dof}dof/meshes/half_arm_2_link.STL" />
-        </geometry>
-      </collision>
-    </link>
-    <joint
-      name="${prefix}joint_3"
-      type="continuous">
-      <origin xyz="0 -0.21038 -0.006375" rpy="-1.5708 1.2326E-32 -2.9122E-16" />
-      <parent
-        link="${prefix}half_arm_1_link" />
-      <child
-        link="${prefix}half_arm_2_link" />
-      <axis
-        xyz="0 0 1" />
-      <limit
-        effort="39"
-        velocity="1.3963" />
-    </joint>
     <link name="${prefix}forearm_link">
       <inertial>
@@ -164,5 +169,6 @@
       <axis
         xyz="0 0 1" />
-      <limit lower="-2.66" upper="2.66" effort="39" velocity="1.3963" />
+        <!-- Changed upper bound from 2.66 to 0 -->
+      <limit lower="-2.66" upper="0.0" effort="39" velocity="1.3963" />
     </joint>
     <link name="${prefix}spherical_wrist_1_link">

File: src/ros_kortex/kortex_description/robots/kortex_robot.xacro (robot description, xacro)
@@ -114,5 +114,5 @@
                 </link>
                 <joint name="${prefix}extrusion_joint" type="fixed">
-                    <origin xyz="0.05 0 -0.024" rpy="0 0 0" />
+                    <origin xyz="-0.05 0 -0.024" rpy="0 0 0" />
                     <parent link="${prefix}kinova_plate_link" />
                     <child link="${prefix}extrusion_link" />

File: src/ros_kortex/kortex_move_it_config/gen3_move_it_config/config/7dof/gen3.srdf.xacro (robot description, xacro)
@@ -38,4 +38,13 @@
         <joint name="$(arg prefix)joint_5" value="0" />
         <joint name="$(arg prefix)joint_6" value="0.96" />
+        <joint name="$(arg prefix)joint_7" value="1.57" />
+    </group_state>
+    <group_state name="horizontal_home" group="arm">
+        <joint name="$(arg prefix)joint_1" value="0" />
+        <joint name="$(arg prefix)joint_2" value="0.26" />
+        <joint name="$(arg prefix)joint_3" value="3.14" />
+        <joint name="$(arg prefix)joint_4" value="-2.27" />
+        <joint name="$(arg prefix)joint_5" value="0" />
+        <joint name="$(arg prefix)joint_6" value="-0.59" />
         <joint name="$(arg prefix)joint_7" value="1.57" />
     </group_state>
@@ -80,4 +89,22 @@
     <disable_collisions link1="$(arg prefix)shoulder_link" link2="$(arg prefix)adapter_link" reason="Never" />
     <disable_collisions link1="$(arg prefix)base_link" link2="$(arg prefix)adapter_link" reason="Never" />
+    <!-- Disable collisions for the bracelet link and all the camera and lense links -->
+    <disable_collisions link1="$(arg prefix)bracelet_link" link2="$(arg prefix)left_camera_link" reason="Never" />
+    <disable_collisions link1="$(arg prefix)bracelet_link" link2="$(arg prefix)right_camera_link" reason="Never" />
+    <disable_collisions link1="$(arg prefix)bracelet_link" link2="$(arg prefix)left_camera_link_lens" reason="Never" />
+    <disable_collisions link1="$(arg prefix)bracelet_link" link2="$(arg prefix)right_camera_link_lens" reason="Never" />
+    <disable_collisions link1="$(arg prefix)bracelet_link" link2="$(arg prefix)left_camera_link_optical" reason="Never" />
+    <disable_collisions link1="$(arg prefix)bracelet_link" link2="$(arg prefix)right_camera_link_optical" reason="Never" />
+    <disable_collisions link1="$(arg prefix)bracelet_link" link2="$(arg prefix)camera_plate_link" reason="Never" />
+    <disable_collisions link1="$(arg prefix)bracelet_link" link2="$(arg prefix)top_plate_link" reason="Never" />
+    <!-- Disable collisions for the spherical wrist 2 link -->
+    <disable_collisions link1="$(arg prefix)spherical_wrist_2_link" link2="$(arg prefix)left_camera_link" reason="Never" />
+    <disable_collisions link1="$(arg prefix)spherical_wrist_2_link" link2="$(arg prefix)right_camera_link" reason="Never" />
+    <disable_collisions link1="$(arg prefix)spherical_wrist_2_link" link2="$(arg prefix)left_camera_link_lens" reason="Never" />
+    <disable_collisions link1="$(arg prefix)spherical_wrist_2_link" link2="$(arg prefix)right_camera_link_lens" reason="Never" />
+    <disable_collisions link1="$(arg prefix)spherical_wrist_2_link" link2="$(arg prefix)left_camera_link_optical" reason="Never" />
+    <disable_collisions link1="$(arg prefix)spherical_wrist_2_link" link2="$(arg prefix)right_camera_link_optical" reason="Never" />
+    <disable_collisions link1="$(arg prefix)spherical_wrist_2_link" link2="$(arg prefix)camera_plate_link" reason="Never" />
+    <disable_collisions link1="$(arg prefix)spherical_wrist_2_link" link2="$(arg prefix)top_plate_link" reason="Never" />
     <!-- Disable collisions for the left camera links and the lenses -->
     <disable_collisions link1="$(arg prefix)left_camera_link" link2="$(arg prefix)left_camera_link_lens" reason="Adjacent" />
@@ -94,4 +121,12 @@
     <disable_collisions link1="$(arg prefix)top_plate_link" link2="$(arg prefix)left_camera_link" reason="Never" />
     <disable_collisions link1="$(arg prefix)top_plate_link" link2="$(arg prefix)right_camera_link" reason="Never" />
+    <!-- Disable collisions between left and right brackets and plates -->
+    <disable_collisions link1="$(arg prefix)left_side_bracket_link" link2="$(arg prefix)top_plate_link" reason="Adjacent" />
+    <disable_collisions link1="$(arg prefix)right_side_bracket_link" link2="$(arg prefix)top_plate_link" reason="Adjacent" />
+    <disable_collisions link1="$(arg prefix)left_side_bracket_link" link2="$(arg prefix)camera_plate_link" reason="Adjacent" />
+    <disable_collisions link1="$(arg prefix)right_side_bracket_link" link2="$(arg prefix)camera_plate_link" reason="Adjacent" />
+    <disable_collisions link1="$(arg prefix)left_side_bracket_link" link2="$(arg prefix)left_camera_link" reason="Adjacent" />
+    <disable_collisions link1="$(arg prefix)right_side_bracket_link" link2="$(arg prefix)right_camera_link" reason="Adjacent" />
+    <disable_collisions link1="$(arg prefix)left_side_bracket_link" link2="$(arg prefix)right_side_bracket_link" reason="Never" />
     <!-- Mounting plate collision disable -->
     <disable_collisions link1="$(arg prefix)mounting_plate_link" link2="$(arg prefix)adapter_link" reason="Never" />
@@ -101,5 +136,7 @@
     <disable_collisions link1="$(arg prefix)spherical_wrist_1_link" link2="$(arg prefix)mounting_plate_link" reason="Never" />
     <disable_collisions link1="$(arg prefix)forearm_link" link2="$(arg prefix)mounting_plate_link" reason="Never" />
-    <disable_collisions link1="$(arg prefix)kinova_plate_link" link2="$(arg prefix)mounting_plate_link" reason="Never" />
+    <disable_collisions link1="$(arg prefix)kinova_plate_link" link2="$(arg prefix)mounting_plate_link" reason="Adjacent" />
+    <disable_collisions link1="$(arg prefix)mounting_plate_link" link2="$(arg prefix)extrusion_link" reason="Never" />
+    <disable_collisions link1="$(arg prefix)kinova_plate_link" link2="$(arg prefix)extrusion_link" reason="Adjacent" />
     <disable_collisions link1="$(arg prefix)forearm_link" link2="$(arg prefix)half_arm_1_link" reason="Never" />
     <disable_collisions link1="$(arg prefix)forearm_link" link2="$(arg prefix)half_arm_2_link" reason="Adjacent" />
