Commit message: Camera URDFS changed for HE calibration

File: src/flir_camera_driver/flir_camera_description/urdf/flir_blackflys.urdf.xacro (robot description, xacro)
@@ -10,5 +10,11 @@
                 lens_r:=0.016 lens_h:=0.04 lens_mass:= 0.05
                 hfov:=1.0471975512 fps:=30 width:=720 height:=540 format:=R8G8B8 near:=0.5 far:=300">
-        <link name="${frame}">
+        <link name="${frame}"/>
+        <joint name="${frame}_body_joint" type="fixed">
+            <origin xyz="0 0 0" rpy="${pi/2} ${-pi/2} 0" />
+            <parent link="${frame}"/>
+            <child link="${frame}_body"/>
+        </joint>
+        <link name="${frame}_body">
         <inertial>
             <mass value="${camera_mass}" />
@@ -54,18 +60,30 @@
         </collision>
         </link>
-        <link name="${frame}_optical" />
         <joint name="${frame}_lens_joint" type="fixed">
         <origin xyz="0.02685 0 0.01425" rpy="0 0 0" />
-        <parent link="${frame}" />
+        <parent link="${frame}_body" />
         <child link="${frame}_lens" />
         </joint>
+        <link name="${frame}_virtual_lens" />
+        <joint name="${frame}_virtual_lens_joint" type="fixed">
+        <origin xyz="${lens_h} 0 0" rpy="${-pi/2} 0 ${-pi/2}" />
+        <parent link="${frame}_lens" />
+        <child link="${frame}_virtual_lens" />
+        </joint>
+        <link name="${frame}_optical" />
         <joint name="${frame}_optical_joint" type="fixed">
         <!-- Change made here compared to original rpy -pi/2 0 -pi/2 -->
-        <origin xyz="${lens_h} 0 0" rpy="${pi/2} 0 ${pi/2}" />
-        <parent link="${frame}_lens" />
+        <origin xyz="0 0 0" rpy="0 0 0" />
+        <parent link="${frame}_virtual_lens" />
         <child link="${frame}_optical" />
         </joint>
+        <link name="${frame}_optical_control_link"/>
+        <joint name="${frame}_optical_control_joint" type="fixed">
+        <origin xyz="0 0 0" rpy="0 0 ${pi}" />
+        <parent link="${frame}_optical" />
+        <child link="${frame}_optical_control_link" />
+        </joint>
         <!-- Gazebo -->
-        <gazebo reference="${frame}_optical">
+        <!-- <gazebo reference="${frame}_optical">
         <material>Gazebo/Grey</material>
         <sensor type="camera" name="${name}">
@@ -104,5 +122,5 @@
             </plugin>
         </sensor>
-        </gazebo>
+        </gazebo> -->
     </xacro:macro>
 </robot>

File: src/ros_kortex/kortex_description/robots/kortex_robot.xacro (robot description, xacro)
@@ -44,12 +44,12 @@
             </joint>
             <!-- Define a joint with the tool frame as a parent called camera_joint -->
-            <joint name="${prefix}camera_joint" type="fixed">
+            <!-- <joint name="${prefix}camera_joint" type="fixed">
                 <origin xyz="0.0 0.1 0.04" rpy="${-pi/2} 0 0" />
                 <parent link="${prefix}tool_frame" />
                 <child link="${prefix}camera_link" />
                 <axis xyz="0 0 0" />
-            </joint>
+            </joint> -->
             <!-- Define camera_link -->
-            <link name="${prefix}camera_link"/>
+            <!-- <link name="${prefix}camera_link"/> -->
             <xacro:if value="${not sim}">
                 <!-- Add mounting plate -->
@@ -240,16 +240,16 @@
                 <!-- Add cameras -->
                 <xacro:include filename="$(find flir_camera_description)/urdf/flir_blackflys.urdf.xacro" />
-                <xacro:flir_blackflys name="left_camera" frame="${prefix}left_camera_link" />
+                <xacro:flir_blackflys name="left_camera" frame="${prefix}left_camera" />
                 <joint name="${prefix}left_camera_joint" type="fixed">
-                    <origin xyz="0.02 0.01565 0" rpy="${pi} 0 ${pi/2}" />
+                    <origin xyz="0.02 0.01565 0" rpy="${-pi/2} ${pi} 0" />
                     <parent link="${prefix}camera_plate_link" />
-                    <child link="${prefix}left_camera_link" />
-                    <axis xyz="0 0 0" />
-                </joint>
-                <xacro:flir_blackflys name="right_camera" frame="${prefix}right_camera_link" />
+                    <child link="${prefix}left_camera" />
+                    <axis xyz="0 0 0" />
+                </joint>
+                <xacro:flir_blackflys name="right_camera" frame="${prefix}right_camera" />
                 <joint name="${prefix}right_camera_joint" type="fixed">
-                    <origin xyz="-0.02 0.01565 0" rpy="${pi} 0 ${pi/2}" />
+                    <origin xyz="-0.02 0.01565 0" rpy="${-pi/2} ${pi} 0" />
                     <parent link="${prefix}camera_plate_link" />
-                    <child link="${prefix}right_camera_link" />
+                    <child link="${prefix}right_camera" />
                     <axis xyz="0 0 0" />
                 </joint>

File: src/ros_kortex/kortex_move_it_config/gen3_move_it_config/config/7dof/gen3.srdf.xacro (robot description, xacro)
@@ -26,6 +26,7 @@
         <joint name="$(arg prefix)camera_plate_joint"/>
         <joint name="$(arg prefix)left_camera_joint"/>
-        <joint name="$(arg prefix)left_camera_link_lens_joint"/>
-        <joint name="$(arg prefix)left_camera_link_optical_joint"/>
+        <joint name="$(arg prefix)left_camera_lens_joint"/>
+        <joint name="$(arg prefix)left_camera_optical_joint"/>
+        <joint name="$(arg prefix)left_camera_optical_control_joint"/>
         <!-- <joint name="$(arg prefix)camera_joint" /> -->
     </group>
@@ -90,35 +91,43 @@
     <disable_collisions link1="$(arg prefix)base_link" link2="$(arg prefix)adapter_link" reason="Never" />
     <!-- Disable collisions for the bracelet link and all the camera and lense links -->
-    <disable_collisions link1="$(arg prefix)bracelet_link" link2="$(arg prefix)left_camera_link" reason="Never" />
-    <disable_collisions link1="$(arg prefix)bracelet_link" link2="$(arg prefix)right_camera_link" reason="Never" />
-    <disable_collisions link1="$(arg prefix)bracelet_link" link2="$(arg prefix)left_camera_link_lens" reason="Never" />
-    <disable_collisions link1="$(arg prefix)bracelet_link" link2="$(arg prefix)right_camera_link_lens" reason="Never" />
-    <disable_collisions link1="$(arg prefix)bracelet_link" link2="$(arg prefix)left_camera_link_optical" reason="Never" />
-    <disable_collisions link1="$(arg prefix)bracelet_link" link2="$(arg prefix)right_camera_link_optical" reason="Never" />
+    <disable_collisions link1="$(arg prefix)bracelet_link" link2="$(arg prefix)left_camera" reason="Never" />
+    <disable_collisions link1="$(arg prefix)bracelet_link" link2="$(arg prefix)right_camera" reason="Never" />
+    <disable_collisions link1="$(arg prefix)bracelet_link" link2="$(arg prefix)left_camera_lens" reason="Never" />
+    <disable_collisions link1="$(arg prefix)bracelet_link" link2="$(arg prefix)right_camera_lens" reason="Never" />
+    <disable_collisions link1="$(arg prefix)bracelet_link" link2="$(arg prefix)left_camera_optical" reason="Never" />
+    <disable_collisions link1="$(arg prefix)bracelet_link" link2="$(arg prefix)right_camera_optical" reason="Never" />
     <disable_collisions link1="$(arg prefix)bracelet_link" link2="$(arg prefix)camera_plate_link" reason="Never" />
     <disable_collisions link1="$(arg prefix)bracelet_link" link2="$(arg prefix)top_plate_link" reason="Never" />
     <!-- Disable collisions for the spherical wrist 2 link -->
-    <disable_collisions link1="$(arg prefix)spherical_wrist_2_link" link2="$(arg prefix)left_camera_link" reason="Never" />
-    <disable_collisions link1="$(arg prefix)spherical_wrist_2_link" link2="$(arg prefix)right_camera_link" reason="Never" />
-    <disable_collisions link1="$(arg prefix)spherical_wrist_2_link" link2="$(arg prefix)left_camera_link_lens" reason="Never" />
-    <disable_collisions link1="$(arg prefix)spherical_wrist_2_link" link2="$(arg prefix)right_camera_link_lens" reason="Never" />
-    <disable_collisions link1="$(arg prefix)spherical_wrist_2_link" link2="$(arg prefix)left_camera_link_optical" reason="Never" />
-    <disable_collisions link1="$(arg prefix)spherical_wrist_2_link" link2="$(arg prefix)right_camera_link_optical" reason="Never" />
+    <disable_collisions link1="$(arg prefix)spherical_wrist_2_link" link2="$(arg prefix)left_camera" reason="Never" />
+    <disable_collisions link1="$(arg prefix)spherical_wrist_2_link" link2="$(arg prefix)right_camera" reason="Never" />
+    <disable_collisions link1="$(arg prefix)spherical_wrist_2_link" link2="$(arg prefix)left_camera_lens" reason="Never" />
+    <disable_collisions link1="$(arg prefix)spherical_wrist_2_link" link2="$(arg prefix)right_camera_lens" reason="Never" />
+    <disable_collisions link1="$(arg prefix)spherical_wrist_2_link" link2="$(arg prefix)left_camera_optical" reason="Never" />
+    <disable_collisions link1="$(arg prefix)spherical_wrist_2_link" link2="$(arg prefix)right_camera_optical" reason="Never" />
     <disable_collisions link1="$(arg prefix)spherical_wrist_2_link" link2="$(arg prefix)camera_plate_link" reason="Never" />
     <disable_collisions link1="$(arg prefix)spherical_wrist_2_link" link2="$(arg prefix)top_plate_link" reason="Never" />
-    <!-- Disable collisions for the left camera links and the lenses -->
-    <disable_collisions link1="$(arg prefix)left_camera_link" link2="$(arg prefix)left_camera_link_lens" reason="Adjacent" />
-    <disable_collisions link1="$(arg prefix)left_camera_link" link2="$(arg prefix)left_camera_link_optical" reason="Adjacent" />
-    <disable_collisions link1="$(arg prefix)left_camera_link_lens" link2="$(arg prefix)left_camera_link_optical" reason="Adjacent" />
-    <!-- Disable collisions for the right camera links and lenses -->
-    <disable_collisions link1="$(arg prefix)right_camera_link" link2="$(arg prefix)right_camera_link_lens" reason="Adjacent" />
-    <disable_collisions link1="$(arg prefix)right_camera_link" link2="$(arg prefix)right_camera_link_optical" reason="Adjacent" />
-    <disable_collisions link1="$(arg prefix)right_camera_link_lens" link2="$(arg prefix)right_camera_link_optical" reason="Adjacent" />
+    <!-- Disable collisions for the left camera links and the lenses and left_camera_body-->
+    <disable_collisions link1="$(arg prefix)left_camera" link2="$(arg prefix)left_camera_lens" reason="Adjacent" />
+    <disable_collisions link1="$(arg prefix)left_camera" link2="$(arg prefix)left_camera_optical" reason="Adjacent" />
+    <disable_collisions link1="$(arg prefix)left_camera_lens" link2="$(arg prefix)left_camera_optical" reason="Adjacent" />
+    <disable_collisions link1="$(arg prefix)left_camera" link2="$(arg prefix)left_camera_body" reason="Adjacent" />
+    <disable_collisions link1="$(arg prefix)left_camera_lens" link2="$(arg prefix)left_camera_body" reason="Adjacent" />
+    <disable_collisions link1="$(arg prefix)left_camera_optical" link2="$(arg prefix)left_camera_body" reason="Adjacent" />
+    <!-- Disable collisions for the right camera links and lenses and right_camera_body-->
+    <disable_collisions link1="$(arg prefix)right_camera" link2="$(arg prefix)right_camera_lens" reason="Adjacent" />
+    <disable_collisions link1="$(arg prefix)right_camera" link2="$(arg prefix)right_camera_optical" reason="Adjacent" />
+    <disable_collisions link1="$(arg prefix)right_camera_lens" link2="$(arg prefix)right_camera_optical" reason="Adjacent" />
+    <disable_collisions link1="$(arg prefix)right_camera" link2="$(arg prefix)right_camera_body" reason="Adjacent" />
+    <disable_collisions link1="$(arg prefix)right_camera_lens" link2="$(arg prefix)right_camera_body" reason="Adjacent" />
+    <disable_collisions link1="$(arg prefix)right_camera_optical" link2="$(arg prefix)right_camera_body" reason="Adjacent" />
     <!-- Disable collisions for the plates and cameras-->
     <disable_collisions link1="$(arg prefix)camera_plate_link" link2="$(arg prefix)top_plate_link" reason="Never" />
-    <disable_collisions link1="$(arg prefix)camera_plate_link" link2="$(arg prefix)left_camera_link" reason="Adjacent" />
-    <disable_collisions link1="$(arg prefix)camera_plate_link" link2="$(arg prefix)right_camera_link" reason="Adjacent" />
-    <disable_collisions link1="$(arg prefix)top_plate_link" link2="$(arg prefix)left_camera_link" reason="Never" />
-    <disable_collisions link1="$(arg prefix)top_plate_link" link2="$(arg prefix)right_camera_link" reason="Never" />
+    <disable_collisions link1="$(arg prefix)camera_plate_link" link2="$(arg prefix)left_camera" reason="Adjacent" />
+    <disable_collisions link1="$(arg prefix)camera_plate_link" link2="$(arg prefix)right_camera" reason="Adjacent" />
+    <disable_collisions link1="$(arg prefix)camera_plate_link" link2="$(arg prefix)left_camera_body" reason="Adjacent" />
+    <disable_collisions link1="$(arg prefix)camera_plate_link" link2="$(arg prefix)right_camera_body" reason="Adjacent" />
+    <disable_collisions link1="$(arg prefix)top_plate_link" link2="$(arg prefix)left_camera" reason="Never" />
+    <disable_collisions link1="$(arg prefix)top_plate_link" link2="$(arg prefix)right_camera" reason="Never" />
     <!-- Disable collisions between left and right brackets and plates -->
     <disable_collisions link1="$(arg prefix)left_side_bracket_link" link2="$(arg prefix)top_plate_link" reason="Adjacent" />
@@ -126,6 +135,8 @@
     <disable_collisions link1="$(arg prefix)left_side_bracket_link" link2="$(arg prefix)camera_plate_link" reason="Adjacent" />
     <disable_collisions link1="$(arg prefix)right_side_bracket_link" link2="$(arg prefix)camera_plate_link" reason="Adjacent" />
-    <disable_collisions link1="$(arg prefix)left_side_bracket_link" link2="$(arg prefix)left_camera_link" reason="Adjacent" />
-    <disable_collisions link1="$(arg prefix)right_side_bracket_link" link2="$(arg prefix)right_camera_link" reason="Adjacent" />
+    <disable_collisions link1="$(arg prefix)left_side_bracket_link" link2="$(arg prefix)left_camera" reason="Adjacent" />
+    <disable_collisions link1="$(arg prefix)right_side_bracket_link" link2="$(arg prefix)right_camera" reason="Adjacent" />
+    <disable_collisions link1="$(arg prefix)left_side_bracket_link" link2="$(arg prefix)left_camera_body" reason="Adjacent" />
+    <disable_collisions link1="$(arg prefix)right_side_bracket_link" link2="$(arg prefix)right_camera_body" reason="Adjacent" />
     <disable_collisions link1="$(arg prefix)left_side_bracket_link" link2="$(arg prefix)right_side_bracket_link" reason="Never" />
     <!-- Mounting plate collision disable -->

Commit message: Handeye calibration added and working

File: src/flir_camera_driver/flir_camera_description/urdf/flir_blackflys.urdf.xacro (robot description, xacro)
@@ -74,5 +74,5 @@
         <joint name="${frame}_optical_joint" type="fixed">
         <!-- Change made here compared to original rpy -pi/2 0 -pi/2 -->
-        <origin xyz="0 0 0" rpy="0 0 0" />
+        <origin xyz="-0.004631252935621712 0.0006080915071296437 -0.013604342613663393" rpy="-0.00824770352247518 -0.06059481072650077 -0.004472121102411795" />
         <parent link="${frame}_virtual_lens" />
         <child link="${frame}_optical" />

Commit message: Updates

File: src/flir_camera_driver/flir_camera_description/urdf/flir_blackflys.urdf.xacro (robot description, xacro)
@@ -74,5 +74,8 @@
         <joint name="${frame}_optical_joint" type="fixed">
         <!-- Change made here compared to original rpy -pi/2 0 -pi/2 -->
-        <origin xyz="-0.004631252935621712 0.0006080915071296437 -0.013604342613663393" rpy="-0.00824770352247518 -0.06059481072650077 -0.004472121102411795" />
+        <origin xyz="0.03675341975118588
+                    0.0011005389185428562
+                    -0.010802901733302936"
+                rpy="0.0008015 -0.0685631 0.008044"/>
         <parent link="${frame}_virtual_lens" />
         <child link="${frame}_optical" />

Commit message: New tracking. Unstable, not cartesian

File: src/flir_camera_driver/flir_camera_description/urdf/flir_blackflys.urdf.xacro (robot description, xacro)
@@ -74,8 +74,8 @@
         <joint name="${frame}_optical_joint" type="fixed">
         <!-- Change made here compared to original rpy -pi/2 0 -pi/2 -->
-        <origin xyz="0.03675341975118588
-                    0.0011005389185428562
-                    -0.010802901733302936"
-                rpy="0.0008015 -0.0685631 0.008044"/>
+        <origin xyz="-0.005250906495466192
+                      0.0020824504039154
+                      0.014754798067452776"
+                rpy="-0.002463045536706444 -0.07124202023637377 0.015601308334355551"/>
         <parent link="${frame}_virtual_lens" />
         <child link="${frame}_optical" />

Commit message: HE_calib

File: src/flir_camera_driver/flir_camera_description/urdf/flir_blackflys.urdf.xacro (robot description, xacro)
@@ -74,8 +74,8 @@
         <joint name="${frame}_optical_joint" type="fixed">
         <!-- Change made here compared to original rpy -pi/2 0 -pi/2 -->
-        <origin xyz="-0.005250906495466192
-                      0.0020824504039154
-                      0.014754798067452776"
-                rpy="-0.002463045536706444 -0.07124202023637377 0.015601308334355551"/>
+        <origin xyz="0.0012889413703012118
+                     0.0006408808146250485
+                    -0.00911597551860998"
+                rpy="0.005898370573761779 -0.08552397363300532 -0.002691160094542855"/>
         <parent link="${frame}_virtual_lens" />
         <child link="${frame}_optical" />
